File: fpv-library/repos/Autonomous-Unmanned-System-An-open-source-Unmanned-Aircraft-System/Flight Controller Hardware/FlightController.kicad_sch (KiCad schematic)
At the start: 38 parts, among them J1 Conn_01x08_Pin, P1 USB_C_Plug_USB2.0, SW1 SW_Push, SW2 SW_Nidec_CAS-120A1, U1 STM32H723ZGIx, U2 AMS1117-3.3, Y1 Crystal_GND24

Commit message: fpv-library: automated discover, triage, sync
Other:
- note added: "<--- BEING USED AS INTERNAL TIMER 10ms timeout"
